Commit message: practice 4

File: src/my_r2d2/urdf/r2d2.urdf.xacro (robot description, xacro)
@@ -232,6 +232,13 @@
     <parent link="box"/>
     <child link="lens"/>
-    <limit effort=1000 lower="${- lensradius}" upper="0" velocity="0.5"/>
+    <limit effort="1000" lower="${- lensradius}" upper="0" velocity="0.5"/>
     <origin xyz="0 0 0"/>
   </joint>
+  <link name="base_footprint">
+  </link>
+  <joint name="basetofootprint" type="fixed">
+    <parent link="base_footprint"/>
+    <child link="base_link"/>
+    <origin xyz="0 0 ${-(0.25 - leglen - (wheeldiam/2 + .05) - wheeldiam/2)}"/>
+  </joint>
 </robot>

Commit message: End of P5, AR tag recognition in RVIZ

File: src/my_r2d2/urdf/r2d2.urdf.xacro (robot description, xacro)
@@ -214,5 +214,5 @@
     <origin xyz="${.707*width+0.04} 0 ${.707*width}"/>
   </joint>
-  <link name="lens">
+  <link name="lense">
     <visual>
       <geometry>
@@ -231,7 +231,14 @@
   <joint name="boxtolens" type="prismatic">
     <parent link="box"/>
-    <child link="lens"/>
+    <child link="lense"/>
     <limit effort="1000" lower="${- lensradius}" upper="0" velocity="0.5"/>
     <origin xyz="0 0 0"/>
+  </joint>
+  <link name="eye">
+  </link>
+  <joint name="eyetolens" type="fixed">
+    <parent link="lense"/>
+    <child link="eye"/>
+    <origin rpy="${pi/2} ${-pi} ${pi/2}"/>
   </joint>
   <link name="base_footprint">
